Commit message: Fix URDF visualization issue: Decimate large meshes for PyBullet rendering
Problem:
- Right leg links (r2-r5) were not rendering in PyBullet GUI
- Root cause: Mesh files had excessive triangle counts (200k-225k triangles)
- PyBullet's batched rendering system hit internal limits with large meshes

Solution:
- Applied quadric edge collapse decimation to reduce mesh complexity
- Reduced large meshes by 60-70% while preserving visual quality
- Standardized all link materials to 'grey' for consistency

Changes:
- models/urdf/hunter.urdf: Updated mesh references and materials
- models/meshes/*.STL: Decimated mesh files for optimal rendering
- models/meshes/*.STL.backup: Original high-resolution meshes preserved
- src/smart_decimate.py: Mesh decimation utility using trimesh
- MESH_DECIMATION_GUIDE.md: Documentation for mesh optimization
- URDF_MESH_UPDATE.md: URDF mesh integration documentation

Mesh Reductions:
- leg_r2/l2: 200k → 80k triangles (60% reduction)
- leg_r3/l3: 225k → 90k triangles (60% reduction)
- leg_r4/l4: 57k → 40k triangles (30% reduction)

Result:
✓ Both legs now render correctly in PyBullet GUI
✓ Reasonable visual quality maintained
✓ Original meshes backed up for future use

🤖 Generated with Claude Code

File: models/urdf/hunter.urdf (robot description, URDF)
Before this commit: robot hunter, 16 links, 15 joints
Links:
- link base_link: geometry collision box size=0.184 0.15 0.2; visual mesh filename=../meshes/base_link.STL
- link leg_l1_link: geometry collision box size=0.06 0.07 0.155; visual mesh filename=../meshes/leg_l1_link.STL
- link leg_l2_link: geometry collision cylinder length=0.146 radius=0.065; visual mesh filename=../meshes/leg_l2_link.STL
- link leg_l3_link: geometry collision box size=0.06 0.25 0.05; visual mesh filename=../meshes/leg_l3_link.STL
- link leg_l4_link: geometry collision box size=0.041 0.25 0.03; visual mesh filename=../meshes/leg_l4_link.STL
- link leg_l5_link: geometry collision box size=0.1001 0.0345 0.0175; visual mesh filename=../meshes/leg_l5_link.STL
- link leg_r1_link: geometry collision box size=0.06 0.07 0.155; visual mesh filename=../meshes/leg_r1_link.STL
- link leg_r2_link: geometry collision cylinder length=0.146 radius=0.065; visual mesh filename=../meshes/leg_r2_link.STL
- link leg_r3_link: geometry collision box size=0.06 0.25 0.05; visual mesh filename=../meshes/leg_r3_link.STL
- link leg_r4_link: geometry collision box size=0.041 0.25 0.03; visual mesh filename=../meshes/leg_r4_link.STL
- link leg_r5_link: geometry collision box size=0.1001 0.0345 0.0175; visual mesh filename=../meshes/leg_r5_link.STL
